File: PCB/Phone_Audio_FM_Transmitter.kicad_sch (KiCad schematic)
At the start: 46 parts, among them J1 Vin, J2 Conn_Coaxial, J3 Conn_Coaxial, J4 USB_B_Micro, J6 Rec, J7 Trans, J8 I2S Test Point, U1 TPS5403, U2 Si4706, U3 Si4711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

Commit message: Changed schematic to reflect final design
Parts:
- removed C12: 0.22uF, Capacitor_SMD:C_0805_2012Metric_Pad1.18x1.45mm_HandSolder, symbol Device:C_Small
- removed C14: 12nF, Capacitor_SMD:C_0805_2012Metric_Pad1.18x1.45mm_HandSolder, symbol Device:C_Small
- removed C15: 0.1uF, Capacitor_SMD:C_0805_2012Metric_Pad1.18x1.45mm_HandSolder, symbol Device:C_Small
- removed C16: 22uF, Capacitor_SMD:C_0805_2012Metric_Pad1.18x1.45mm_HandSolder, symbol Device:C_Small
- removed C18, C19: 22pF, Capacitor_SMD:C_0805_2012Metric_Pad1.18x1.45mm_HandSolder, symbol Device:C_Small
- removed D2: D_Schottky, Diode_SMD:D_1206_3216Metric_Pad1.42x1.75mm_HandSolder, symbol Device:D_Schottky
- removed L3: 13uH, Inductor_SMD:L_0805_2012Metric_Pad1.15x1.40mm_HandSolder, symbol Device:L_Small
- removed R11: 82k, Resistor_SMD:R_0805_2012Metric_Pad1.20x1.40mm_HandSolder, symbol Device:R
- removed R12: 2.2k, Resistor_SMD:R_0805_2012Metric_Pad1.20x1.40mm_HandSolder, symbol Device:R
- removed R9: 0, Resistor_SMD:R_0805_2012Metric_Pad1.20x1.40mm_HandSolder, symbol Device:R
- removed U1: TPS5403, Package_SO:SOIC-8_3.9x4.9mm_P1.27mm, symbol Regulator_Switching:TPS5403
- removed Y1: 32.768kHz, Crystal:Crystal_SMD_2012-2Pin_2.0x1.2mm_HandSoldering, symbol Device:Crystal
- added U1: NCP1117-3.3_TO252, Package_TO_SOT_SMD:TO-252-2, symbol Regulator_Linear:NCP1117-3.3_TO252
Connections:
- net TRCLK is gone; now on net RCLK: U3.9 (RCLK), U6.28 (IO17)
- net +3.3V: now also U1.2 (VO)
- net GND: now also U1.1 (GND)
- net RXDO: now also U7.26 (TXD); no longer U7.25 (RXD)
- net TXDO: now also U7.25 (RXD); no longer U7.26 (TXD)
- net at C13.1, J1.1 (Pin_1): now also U1.3 (VI)
- net RRCLK renamed RCLK
Other:
- note added: "Programming"
- moved on the sheet: C13, C2, D1, J1, J3, J7, J8, L2, R10, R4, R5, R8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
